Commit message: Preped world

File: resources/5DOF_Scara/robot.urdf (robot description, URDF)
Before this commit: robot 5DOF_SCARA, 6 links, 5 joints
Links:
- link link4: geometry visual box size=0.05 0.05 0.05; visual cylinder length=0.05 radius=0.06

Commit message: Added inertia and collision properties to robot

File: resources/5DOF_Scara/robot.urdf (robot description, URDF)
Before this commit: robot 5DOF_SCARA, 6 links, 5 joints
Links:
- link link3: mass 1 -> 0.5
- link link4: mass 1 -> 0.1; geometry collision box size=0.05 0.05 0.05; visual box size=0.05 0.05 0.05

Commit message: Graphics mods

File: resources/5DOF_Scara/robot.urdf (robot description, URDF)
Before this commit: robot 5DOF_SCARA, 6 links, 5 joints
Links:
- link base_link: geometry visual cylinder length=0.6 radius=0.1
- link link0: geometry visual cylinder length=1.05 radius=0.07
